File: schematics/alu-test.sch (KiCad schematic (older format))
At the start: 14 parts

Commit message: ALU appears to work as expected
Parts:
- renumbered V8 to V10, V9 to V11, V4 to V12, V6 to V13, V7 to V14, V10 to V2, V2 to V3, V11 to V4, V3 to V5, V12 to V6, V14 to V7, V5 to V8, V13 to V9
Changed lines of the file:
@@
 $EndSheet
 $Comp
-L pspice:VSOURCE V14
+L pspice:VSOURCE V7
 U 1 1 5C552322
 P 10200 3300
-F 0 "V14" V 10565 3300 50  0000 C CNN
+F 0 "V7" V 10565 3300 50  0000 C CNN
 F 1 "dc 5" V 10474 3300 50  0000 C CNN
 F 2 "" H 10200 3300 50  0001 C CNN
@@
 $EndComp
 $Comp
-L pspice:0 #GND014
+L pspice:0 #GND07
 U 1 1 5C5523C6
 P 10800 3300
-F 0 "#GND014" H 10800 3200 50  0001 C CNN
+F 0 "#GND07" H 10800 3200 50  0001 C CNN
 F 1 "0" V 10800 3341 50  0000 L CNN
 F 2 "" H 10800 3300 50  0001 C CNN
@@
 	850  1000 1150 1000
 $Comp
-L pspice:VSOURCE V2
+L pspice:VSOURCE V3
 U 1 1 5C552B09
 P 1450 1800
-F 0 "V2" V 1815 1800 50  0000 C CNN
+F 0 "V3" V 1815 1800 50  0000 C CNN
 F 1 "dc 5" V 1724 1800 50  0000 C CNN
 F 2 "" H 1450 1800 50  0001 C CNN
@@
 $EndComp
 $Comp
-L pspice:0 #GND02
+L pspice:0 #GND03
 U 1 1 5C552B10
 P 850 1800
-F 0 "#GND02" H 850 1700 50  0001 C CNN
+F 0 "#GND03" H 850 1700 50  0001 C CNN
 F 1 "0" V 850 1841 50  0000 L CNN
 F 2 "" H 850 1800 50  0001 C CNN
@@
 	850  1800 1150 1800
 $Comp
-L pspice:VSOURCE V3
+L pspice:VSOURCE V5
 U 1 1 5C552C0D
 P 1450 2600
-F 0 "V3" V 1815 2600 50  0000 C CNN
+F 0 "V5" V 1815 2600 50  0000 C CNN
 F 1 "dc 5" V 1724 2600 50  0000 C CNN
 F 2 "" H 1450 2600 50  0001 C CNN
@@
 $EndComp
 $Comp
-L pspice:0 #GND03
+L pspice:0 #GND05
 U 1 1 5C552C14
 P 850 2600
-F 0 "#GND03" H 850 2500 50  0001 C CNN
+F 0 "#GND05" H 850 2500 50  0001 C CNN
 F 1 "0" V 850 2641 50  0000 L CNN
 F 2 "" H 850 2600 50  0001 C CNN
@@
 	850  2600 1150 2600
 $Comp
-L pspice:VSOURCE V5
+L pspice:VSOURCE V8
 U 1 1 5C552D38
 P 1500 3450
-F 0 "V5" V 1865 3450 50  0000 C CNN
+F 0 "V8" V 1865 3450 50  0000 C CNN
 F 1 "dc 5" V 1774 3450 50  0000 C CNN
 F 2 "" H 1500 3450 50  0001 C CNN
@@
 $EndComp
 $Comp
-L pspice:0 #GND04
+L pspice:0 #GND08
 U 1 1 5C552D3F
 P 900 3450
-F 0 "#GND04" H 900 3350 50  0001 C CNN
+F 0 "#GND08" H 900 3350 50  0001 C CNN
 F 1 "0" V 900 3491 50  0000 L CNN
 F 2 "" H 900 3450 50  0001 C CNN
@@
 	900  3450 1200 3450
 $Comp
-L pspice:VSOURCE V10
+L pspice:VSOURCE V2
 U 1 1 5C553451
 P 5200 1000
-F 0 "V10" V 5565 1000 50  0000 C CNN
+F 0 "V2" V 5565 1000 50  0000 C CNN
 F 1 "dc 5" V 5474 1000 50  0000 C CNN
 F 2 "" H 5200 1000 50  0001 C CNN
@@
 $EndComp
 $Comp
-L pspice:0 #GND09
+L pspice:0 #GND02
 U 1 1 5C553458
 P 4600 1000
-F 0 "#GND09" H 4600 900 50  0001 C CNN
+F 0 "#GND02" H 4600 900 50  0001 C CNN
 F 1 "0" V 4600 1041 50  0000 L CNN
 F 2 "" H 4600 1000 50  0001 C CNN
@@
 	4600 1000 4900 1000
 $Comp
-L pspice:VSOURCE V11
+L pspice:VSOURCE V4
 U 1 1 5C55345F
 P 5200 1800
-F 0 "V11" V 5565 1800 50  0000 C CNN
+F 0 "V4" V 5565 1800 50  0000 C CNN
 F 1 "dc 5" V 5474 1800 50  0000 C CNN
 F 2 "" H 5200 1800 50  0001 C CNN
@@
 $EndComp
 $Comp
-L pspice:0 #GND010
+L pspice:0 #GND04
 U 1 1 5C553466
 P 4600 1800
-F 0 "#GND010" H 4600 1700 50  0001 C CNN
+F 0 "#GND04" H 4600 1700 50  0001 C CNN
 F 1 "0" V 4600 1841 50  0000 L CNN
 F 2 "" H 4600 1800 50  0001 C CNN
@@
 	4600 1800 4900 1800
 $Comp
-L pspice:VSOURCE V12
+L pspice:VSOURCE V6
 U 1 1 5C55346D
 P 5200 2600
-F 0 "V12" V 5565 2600 50  0000 C CNN
+F 0 "V6" V 5565 2600 50  0000 C CNN
 F 1 "dc 5" V 5474 2600 50  0000 C CNN
 F 2 "" H 5200 2600 50  0001 C CNN
@@
 $EndComp
 $Comp
-L pspice:0 #GND011
+L pspice:0 #GND06
 U 1 1 5C553474
 P 4600 2600
-F 0 "#GND011" H 4600 2500 50  0001 C CNN
+F 0 "#GND06" H 4600 2500 50  0001 C CNN
 F 1 "0" V 4600 2641 50  0000 L CNN
 F 2 "" H 4600 2600 50  0001 C CNN
@@
 	4600 2600 4900 2600
 $Comp
-L pspice:VSOURCE V13
+L pspice:VSOURCE V9
 U 1 1 5C55347B
 P 5250 3450
-F 0 "V13" V 5615 3450 50  0000 C CNN
+F 0 "V9" V 5615 3450 50  0000 C CNN
 F 1 "dc 5" V 5524 3450 50  0000 C CNN
 F 2 "" H 5250 3450 50  0001 C CNN
@@
 $EndComp
 $Comp
-L pspice:0 #GND012
+L pspice:0 #GND09
 U 1 1 5C553482
 P 4650 3450
-F 0 "#GND012" H 4650 3350 50  0001 C CNN
+F 0 "#GND09" H 4650 3350 50  0001 C CNN
 F 1 "0" V 4650 3491 50  0000 L CNN
 F 2 "" H 4650 3450 50  0001 C CNN
@@
 	4650 3450 4950 3450
 $Comp
-L pspice:VSOURCE V4
+L pspice:VSOURCE V12
 U 1 1 5C553A22
 P 1450 6600
-F 0 "V4" V 1815 6600 50  0000 C CNN
+F 0 "V12" V 1815 6600 50  0000 C CNN
 F 1 "dc 5" V 1724 6600 50  0000 C CNN
 F 2 "" H 1450 6600 50  0001 C CNN
@@
 $EndComp
 $Comp
-L pspice:0 #GND05
+L pspice:0 #GND012
 U 1 1 5C553A29
 P 1450 7200
-F 0 "#GND05" H 1450 7100 50  0001 C CNN
+F 0 "#GND012" H 1450 7100 50  0001 C CNN
 F 1 "0" V 1450 7241 50  0000 L CNN
 F 2 "" H 1450 7200 50  0001 C CNN
@@
 	1450 7200 1450 6900
 $Comp
-L pspice:VSOURCE V6
+L pspice:VSOURCE V13
 U 1 1 5C553A30
 P 2250 6600
-F 0 "V6" V 2615 6600 50  0000 C CNN
+F 0 "V13" V 2615 6600 50  0000 C CNN
 F 1 "dc 5" V 2524 6600 50  0000 C CNN
 F 2 "" H 2250 6600 50  0001 C CNN
@@
 $EndComp
 $Comp
-L pspice:0 #GND06
+L pspice:0 #GND013
 U 1 1 5C553A37
 P 2250 7200
-F 0 "#GND06" H 2250 7100 50  0001 C CNN
+F 0 "#GND013" H 2250 7100 50  0001 C CNN
 F 1 "0" V 2250 7241 50  0000 L CNN
 F 2 "" H 2250 7200 50  0001 C CNN
@@
 	2250 7200 2250 6900
 $Comp
-L pspice:VSOURCE V7
+L pspice:VSOURCE V14
 U 1 1 5C553A3E
 P 3050 6600
-F 0 "V7" V 3415 6600 50  0000 C CNN
+F 0 "V14" V 3415 6600 50  0000 C CNN
 F 1 "dc 5" V 3324 6600 50  0000 C CNN
 F 2 "" H 3050 6600 50  0001 C CNN
@@
 $EndComp
 $Comp
-L pspice:0 #GND07
+L pspice:0 #GND014
 U 1 1 5C553A45
 P 3050 7200
-F 0 "#GND07" H 3050 7100 50  0001 C CNN
+F 0 "#GND014" H 3050 7100 50  0001 C CNN
 F 1 "0" V 3050 7241 50  0000 L CNN
 F 2 "" H 3050 7200 50  0001 C CNN
@@
 	3050 7200 3050 6900
 $Comp
-L pspice:VSOURCE V8
+L pspice:VSOURCE V10
 U 1 1 5C553A4C
 P 3900 6550
-F 0 "V8" V 4265 6550 50  0000 C CNN
+F 0 "V10" V 4265 6550 50  0000 C CNN
 F 1 "dc 5" V 4174 6550 50  0000 C CNN
 F 2 "" H 3900 6550 50  0001 C CNN
@@
 $EndComp
 $Comp
-L pspice:0 #GND08
+L pspice:0 #GND010
 U 1 1 5C553A53
 P 3900 7150
-F 0 "#GND08" H 3900 7050 50  0001 C CNN
+F 0 "#GND010" H 3900 7050 50  0001 C CNN
 F 1 "0" V 3900 7191 50  0000 L CNN
 F 2 "" H 3900 7150 50  0001 C CNN
@@
 	3900 7150 3900 6850
 $Comp
-L pspice:VSOURCE V9
+L pspice:VSOURCE V11
 U 1 1 5C5548A9
 P 4750 6550
-F 0 "V9" V 5115 6550 50  0000 C CNN
+F 0 "V11" V 5115 6550 50  0000 C CNN
 F 1 "dc 5" V 5024 6550 50  0000 C CNN
 F 2 "" H 4750 6550 50  0001 C CNN
@@
 	4750 7150 4750 6850
 $Comp
-L pspice:0 #GND013
+L pspice:0 #GND011
 U 1 1 5C555094
 P 4750 7150
-F 0 "#GND013" H 4750 7050 50  0001 C CNN
+F 0 "#GND011" H 4750 7050 50  0001 C CNN
 F 1 "0" V 4750 7191 50  0000 L CNN
 F 2 "" H 4750 7150 50  0001 C CNN
