File: schematics/multiplexer-4-4-1-test.sch (KiCad schematic (older format))
At the start: 10 parts

Commit message: Adds ALU Schematics (#1)
* Adds a test for the 4-4-1 multiplexer
* Adds an xor gate
* Updates gitignore to include common swap files and data output
* Adds a four bit bitwise inverter
* Adds a one bit buffer
* Adds a 1->4 bit replicator
* Adds a 4 bit and gate
* ALU is sketched but has functional defects
* Adds a netlist "optimizer" which shortens names for better output parsing
* Adds a simple spice runner
* Adds a model injector and an op test injector
* Basic unit test automation framework for async circuits
* Adds a primitive directory iterator
* Adds some tests for and-2, nor-2, nor-3
* More testing.  Trying to find defect in ALU
* ALU appears to work as expected
* Updates README, adds some ALU tests
* Updates the schematics' README
Parts:
- added V10, V11, V12, V13, V14, V15, V16, V17, V19: dc 5, symbol pspice:VSOURCE
- gave numbers to parts that had none: 10
Connections:
- net labels added: C1in, C2in, C3in, C4in, D1in, D2in, D3in, D4in, S1in, S2in
- net labels removed: SelIn
- wire segments 42 -> 103
Other:
- moved on the sheet: V1, V18, V2, V3, V4, V5, V6, V7, V8, V9
