File: schematics/adder-1-test.sch (KiCad schematic (older format))
At the start: 4 parts

Commit message: Adds ALU Schematics (#1)
* Adds a test for the 4-4-1 multiplexer
* Adds an xor gate
* Updates gitignore to include common swap files and data output
* Adds a four bit bitwise inverter
* Adds a one bit buffer
* Adds a 1->4 bit replicator
* Adds a 4 bit and gate
* ALU is sketched but has functional defects
* Adds a netlist "optimizer" which shortens names for better output parsing
* Adds a simple spice runner
* Adds a model injector and an op test injector
* Basic unit test automation framework for async circuits
* Adds a primitive directory iterator
* Adds some tests for and-2, nor-2, nor-3
* More testing.  Trying to find defect in ALU
* ALU appears to work as expected
* Updates README, adds some ALU tests
* Updates the schematics' README
Parts:
- V2: value PULSE(5 0 2NS 2NS 2NS 50NS 100NS) -> dc 5
- V3: value PULSE(5 0 2NS 2NS 2NS 100NS 200NS) -> dc 5
- V4: value PULSE(5 0 2NS 2NS 2NS 200NS 400NS) -> dc 5
Connections:
- net adder-1/A renamed Ain
- net adder-1/B renamed Bin
- net adder-1/Cin renamed Cin
Changed lines of the file:
@@
 EESchema Schematic File Version 4
+LIBS:adder-1-test-cache
 EELAYER 26 0
 EELAYER END
@@
 P 6250 4450
 F 0 "V2" H 6478 4496 50  0000 L CNN
-F 1 "PULSE(5 0 2NS 2NS 2NS 50NS 100NS)" H 6478 4405 50  0000 L CNN
+F 1 "dc 5" H 6478 4405 50  0000 L CNN
 F 2 "" H 6250 4450 50  0001 C CNN
 F 3 "~" H 6250 4450 50  0001 C CNN
@@
 P 6850 4950
 F 0 "V3" H 7078 4996 50  0000 L CNN
-F 1 "PULSE(5 0 2NS 2NS 2NS 100NS 200NS)" H 7078 4905 50  0000 L CNN
+F 1 "dc 5" H 7078 4905 50  0000 L CNN
 F 2 "" H 6850 4950 50  0001 C CNN
 F 3 "~" H 6850 4950 50  0001 C CNN
@@
 P 7400 5500
 F 0 "V4" H 7628 5546 50  0000 L CNN
-F 1 "PULSE(5 0 2NS 2NS 2NS 200NS 400NS)" H 7628 5455 50  0000 L CNN
+F 1 "dc 5" H 7628 5455 50  0000 L CNN
 F 2 "" H 7400 5500 50  0001 C CNN
 F 3 "~" H 7400 5500 50  0001 C CNN
@@
 Wire Wire Line
 	6750 4150 6250 4150
+Text HLabel 8200 3400 2    50   Input ~ 0
+S
+Wire Wire Line
+	8200 3400 7850 3400
+Text Label 7950 3400 0    50   ~ 0
+Sout
+Text Label 6450 4150 0    50   ~ 0
+Ain
+Text Label 6850 4250 0    50   ~ 0
+Bin
+Text Label 7400 4250 0    50   ~ 0
+Cin
 $EndSCHEMATC

Commit message: Can now automate transient analysis
Parts:
- V1, V2, V3, V4: footprint (none) -> Power_Integrations:PDIP-8
Changed lines of the file:
@@
 $EndDescr
 $Comp
-L pspice:0 #GND0101
+L pspice:0 #GND01
 U 1 1 5C40CC44
 P 6050 3900
-F 0 "#GND0101" H 6050 3800 50  0001 C CNN
+F 0 "#GND01" H 6050 3800 50  0001 C CNN
 F 1 "0" H 6050 3987 50  0000 C CNN
 F 2 "" H 6050 3900 50  0001 C CNN
@@
 F 0 "V1" H 6278 3296 50  0000 L CNN
 F 1 "dc 5" H 6278 3205 50  0000 L CNN
-F 2 "" H 6050 3250 50  0001 C CNN
+F 2 "Power_Integrations:PDIP-8" H 6050 3250 50  0001 C CNN
 F 3 "~" H 6050 3250 50  0001 C CNN
 	1    6050 3250
@@
 Connection ~ 6050 3550
 $Comp
-L pspice:0 #GND0102
+L pspice:0 #GND02
 U 1 1 5C40CEC1
 P 6250 5000
-F 0 "#GND0102" H 6250 4900 50  0001 C CNN
+F 0 "#GND02" H 6250 4900 50  0001 C CNN
 F 1 "0" H 6250 5087 50  0000 C CNN
 F 2 "" H 6250 5000 50  0001 C CNN
@@
 F 0 "V2" H 6478 4496 50  0000 L CNN
 F 1 "dc 5" H 6478 4405 50  0000 L CNN
-F 2 "" H 6250 4450 50  0001 C CNN
+F 2 "Power_Integrations:PDIP-8" H 6250 4450 50  0001 C CNN
 F 3 "~" H 6250 4450 50  0001 C CNN
 	1    6250 4450
@@
 	6250 4750 6250 5000
 $Comp
-L pspice:0 #GND0103
+L pspice:0 #GND03
 U 1 1 5C40D375
 P 6850 5500
-F 0 "#GND0103" H 6850 5400 50  0001 C CNN
+F 0 "#GND03" H 6850 5400 50  0001 C CNN
 F 1 "0" H 6850 5587 50  0000 C CNN
 F 2 "" H 6850 5500 50  0001 C CNN
@@
 F 0 "V3" H 7078 4996 50  0000 L CNN
 F 1 "dc 5" H 7078 4905 50  0000 L CNN
-F 2 "" H 6850 4950 50  0001 C CNN
+F 2 "Power_Integrations:PDIP-8" H 6850 4950 50  0001 C CNN
 F 3 "~" H 6850 4950 50  0001 C CNN
 	1    6850 4950
@@
 	6850 5250 6850 5500
 $Comp
-L pspice:0 #GND0104
+L pspice:0 #GND04
 U 1 1 5C40D430
 P 7400 6050
-F 0 "#GND0104" H 7400 5950 50  0001 C CNN
+F 0 "#GND04" H 7400 5950 50  0001 C CNN
 F 1 "0" H 7400 6137 50  0000 C CNN
 F 2 "" H 7400 6050 50  0001 C CNN
@@
 F 0 "V4" H 7628 5546 50  0000 L CNN
 F 1 "dc 5" H 7628 5455 50  0000 L CNN
-F 2 "" H 7400 5500 50  0001 C CNN
+F 2 "Power_Integrations:PDIP-8" H 7400 5500 50  0001 C CNN
 F 3 "~" H 7400 5500 50  0001 C CNN
 	1    7400 5500
