File: schematics/flip-flop-d-test.sch (KiCad schematic (older format))
At the start: 3 parts

Commit message: Can now automate transient analysis
Connections:
- net flip-flop-d/CLK renamed ClkIn
- net flip-flop-d/D renamed Din
Changed lines of the file:
@@
 $EndDescr
 $Comp
-L pspice:0 #GND0101
+L pspice:0 #GND01
 U 1 1 5C3FF203
 P 3400 3150
-F 0 "#GND0101" H 3400 3050 50  0001 C CNN
+F 0 "#GND01" H 3400 3050 50  0001 C CNN
 F 1 "0" H 3400 3237 50  0000 C CNN
 F 2 "" H 3400 3150 50  0001 C CNN
@@
 F3 "Gnd" I L 4450 2100 50
 F4 "D" I L 4450 2250 50
-F5 "CLK" I L 4450 2350 50
+F5 "Clk" I L 4450 2350 50
 F6 "Q" I R 5150 2350 50
 F7 "NQ" I R 5150 2000 50
@@
 Connection ~ 3400 2600
 $Comp
-L pspice:0 #GND0102
+L pspice:0 #GND02
 U 1 1 5C3FF6A2
 P 3850 3700
-F 0 "#GND0102" H 3850 3600 50  0001 C CNN
+F 0 "#GND02" H 3850 3600 50  0001 C CNN
 F 1 "0" H 3850 3787 50  0000 C CNN
 F 2 "" H 3850 3700 50  0001 C CNN
@@
 	3850 3550 3850 3700
 $Comp
-L pspice:0 #GND0103
+L pspice:0 #GND03
 U 1 1 5C3FF939
 P 4600 3700
-F 0 "#GND0103" H 4600 3600 50  0001 C CNN
+F 0 "#GND03" H 4600 3600 50  0001 C CNN
 F 1 "0" H 4600 3787 50  0000 C CNN
 F 2 "" H 4600 3700 50  0001 C CNN
@@
 Wire Wire Line
 	4400 2950 4600 2950
+Text Label 4400 2700 0    50   ~ 0
+ClkIn
+Text Label 3850 2800 0    50   ~ 0
+Din
+Text HLabel 5400 2000 2    50   Input ~ 0
+NQ
+Wire Wire Line
+	5400 2000 5150 2000
+Text HLabel 5400 2350 2    50   Input ~ 0
+Q
+Wire Wire Line
+	5400 2350 5150 2350
+Text Label 5250 2000 0    50   ~ 0
+NQ
+Text Label 5250 2350 0    50   ~ 0
+Q
 $EndSCHEMATC
